File: power_reg.kicad_sch (KiCad schematic)
At the start: 11 parts, among them U2 AZ1117-3.3, U4 AP2112K-1.8

Commit message: start layout
Parts:
- removed C12: 100nF, Capacitor_SMD:C_0603_1608Metric, symbol Device:C_Small
- removed C9: 10uF, Capacitor_SMD:C_0805_2012Metric, symbol Device:C_Small
Changed lines of the file:
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@@
   (junction (at 93.98 38.1) (diameter 0) (color 0 0 0 0)
   )
-  (junction (at 33.02 35.56) (diameter 0) (color 0 0 0 0)
-  )
   (junction (at 35.56 35.56) (diameter 0) (color 0 0 0 0)
   )
@@
   (junction (at 53.34 35.56) (diameter 0) (color 0 0 0 0)
   )
-  (junction (at 33.02 45.72) (diameter 0) (color 0 0 0 0)
-  )
-  (junction (at 38.1 35.56) (diameter 0) (color 0 0 0 0)
-  )
   (wire (pts (xy 46.99 35.56) (xy 53.34 35.56))
     (stroke (width 0) (type default))
   )
-  (wire (pts (xy 33.02 35.56) (xy 33.02 39.37))
-    (stroke (width 0) (type default))
-  )
-  (wire (pts (xy 38.1 35.56) (xy 38.1 39.37))
-    (stroke (width 0) (type default))
-  )
-  (wire (pts (xy 38.1 35.56) (xy 39.37 35.56))
-    (stroke (width 0) (type default))
-  )
   (wire (pts (xy 56.515 38.1) (xy 58.42 38.1))
     (stroke (width 0) (type default))
@@
     (stroke (width 0) (type default))
   )
-  (wire (pts (xy 38.1 44.45) (xy 38.1 45.72))
-    (stroke (width 0) (type default))
-  )
   (wire (pts (xy 55.88 68.58) (xy 60.96 68.58))
     (stroke (width 0) (type default))
   )
-  (wire (pts (xy 33.02 44.45) (xy 33.02 45.72))
-    (stroke (width 0) (type default))
-  )
-  (wire (pts (xy 35.56 35.56) (xy 38.1 35.56))
+  (wire (pts (xy 35.56 35.56) (xy 39.37 35.56))
     (stroke (width 0) (type default))
   )
@@
     (stroke (width 0) (type default))
   )
-  (wire (pts (xy 33.02 45.72) (xy 38.1 45.72))
-    (stroke (width 0) (type default))
-  )
-  (wire (pts (xy 33.02 45.72) (xy 33.02 46.99))
-    (stroke (width 0) (type default))
-  )
   (wire (pts (xy 60.96 71.12) (xy 60.96 68.58))
     (stroke (width 0) (type default))
   )
-  (wire (pts (xy 30.48 35.56) (xy 33.02 35.56))
-    (stroke (width 0) (type default))
-  )
-  (wire (pts (xy 33.02 35.56) (xy 35.56 35.56))
+  (wire (pts (xy 30.48 35.56) (xy 35.56 35.56))
     (stroke (width 0) (type default))
   )
@@
     )
   )
-  (symbol (lib_id "Device:C_Small") (at 38.1 41.91 0) (unit 1)
-    (in_bom yes) (on_board yes) (dnp yes) (fields_autoplaced)
-    (property "Reference" "C12" (at 40.4241 40.7042 0)
-      (effects (font (size 1.27 1.27)) (justify left))
-    )
-    (property "Value" "100nF" (at 40.4241 43.1284 0)
-      (effects (font (size 1.27 1.27)) (justify left))
-    )
-    (property "Footprint" "Capacitor_SMD:C_0603_1608Metric" (at 38.1 41.91 0)
-      (effects (font (size 1.27 1.27)) hide)
-    )
-    (property "Datasheet" "~" (at 38.1 41.91 0)
-      (effects (font (size 1.27 1.27)) hide)
-    )
-    (property "JLC" "" (at 38.1 41.91 0)
-      (effects (font (size 1.27 1.27)) hide)
-    )
-    (property "Part number" "" (at 38.1 41.91 0)
-      (effects (font (size 1.27 1.27)) hide)
-    )
-    (property "MPN" "" (at 38.1 41.91 0)
-      (effects (font (size 1.27 1.27)) hide)
-    )
-    (pin "1")
-    (pin "2")
-    (instances
-      (project "mpw-mb1"
-        (path "/20adca1d-43a1-4784-9682-8b7dd1c7d330"
-          (reference "C12") (unit 1)
-        )
-      )
-      (project "tt-vga-clock"
-        (path "/d2f3109e-08ec-4d18-8cdf-c360e3b1458b"
-          (reference "C5") (unit 1)
-        )
-        (path "/d2f3109e-08ec-4d18-8cdf-c360e3b1458b/f16a8f72-c85c-4194-9580-d5ee14eb71ec"
-          (reference "C17") (unit 1)
-        )
-      )
-    )
-  )
   (symbol (lib_id "power:+5V") (at 53.34 33.02 0) (unit 1)
     (in_bom yes) (on_board yes) (dnp no) (fields_autoplaced)
@@
         (path "/d2f3109e-08ec-4d18-8cdf-c360e3b1458b/f16a8f72-c85c-4194-9580-d5ee14eb71ec"
           (reference "#FLG02") (unit 1)
-        )
-      )
-    )
-  )
-  (symbol (lib_id "Device:C_Small") (at 33.02 41.91 0) (mirror y) (unit 1)
-    (in_bom yes) (on_board yes) (dnp yes)
-    (property "Reference" "C9" (at 30.6959 40.7042 0)
-      (effects (font (size 1.27 1.27)) (justify left))
-    )
-    (property "Value" "10uF" (at 30.6959 43.1284 0)
-      (effects (font (size 1.27 1.27)) (justify left))
-    )
-    (property "Footprint" "Capacitor_SMD:C_0805_2012Metric" (at 33.02 41.91 0)
-      (effects (font (size 1.27 1.27)) hide)
-    )
-    (property "Datasheet" "~" (at 33.02 41.91 0)
-      (effects (font (size 1.27 1.27)) hide)
-    )
-    (property "JLC" "" (at 33.02 41.91 0)
-      (effects (font (size 1.27 1.27)) hide)
-    )
-    (property "Part number" "" (at 33.02 41.91 0)
-      (effects (font (size 1.27 1.27)) hide)
-    )
-    (property "MPN" "" (at 33.02 41.91 0)
-      (effects (font (size 1.27 1.27)) hide)
-    )
-    (pin "1")
-    (pin "2")
-    (instances
-      (project "mpw-mb1"
-        (path "/20adca1d-43a1-4784-9682-8b7dd1c7d330"
-          (reference "C9") (unit 1)
-        )
-      )
-      (project "tt-vga-clock"
-        (path "/d2f3109e-08ec-4d18-8cdf-c360e3b1458b"
-          (reference "C2") (unit 1)
-        )
-        (path "/d2f3109e-08ec-4d18-8cdf-c360e3b1458b/f16a8f72-c85c-4194-9580-d5ee14eb71ec"
-          (reference "C16") (unit 1)
         )
       )
@@
         )
       )
-    )
-  )
-  (symbol (lib_id "power:GND") (at 33.02 46.99 0) (unit 1)
-    (in_bom yes) (on_board yes) (dnp no)
-    (property "Reference" "#PWR032" (at 33.02 53.34 0)
-      (effects (font (size 1.27 1.27)) hide)
-    )
-    (property "Value" "GND" (at 33.02 50.8 0)
-      (effects (font (size 1.27 1.27)))
-    )
-    (property "Footprint" "" (at 33.02 46.99 0)
-      (effects (font (size 1.27 1.27)) hide)
-    )
-    (property "Datasheet" "" (at 33.02 46.99 0)
-      (effects (font (size 1.27 1.27)) hide)
-    )
-    (pin "1")
-    (instances
-      (project "mpw-mb1"
-        (path "/20adca1d-43a1-4784-9682-8b7dd1c7d330"
-          (reference "#PWR032") (unit 1)
-        )
-      )
-      (project "tt-vga-clock"
-        (path "/d2f3109e-08ec-4d18-8cdf-c360e3b1458b"
-          (reference "#PWR02") (unit 1)
-        )
-        (path "/d2f3109e-08ec-4d18-8cdf-c360e3b1458b/f16a8f72-c85c-4194-9580-d5ee14eb71ec"
-          (reference "#PWR070") (unit 1)
-        )
-      )
